File: KiCad/LibrePulse.kicad_sch (KiCad schematic)
At the start: 118 parts, among them IC1 TPS62841YBGR, IC2 BQ21088YBGR, IC3 AS6221, IC4 BME690, IC5 ICU-10201, IC6 KLMCG4JETD-B041, IC7 OPT3007YMFR, J1 Micro_SD_Card, M1 VLV041235L, U1 AS7058, U10 TPSM81299VCMR, U11 ESP32-P4NRW32, U12 BMI270, U13 PCAL6416AHF, U14 BMM350, U15 DRV2605LDGS, U16 MAX98357A, U17 W25Q128JVE, U18 LM3643YFFR, U19 ESP32-C3, U2 ET020AM03-HT, U20 ASGPDF254_A, U3 RV-3028-C8-32.768KHZ-1PPM-TA-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, U4 MS5837-30BA, U5 BQ27427YZFR, U6 BQ51013CQWRHLRQ1, U7 AS7331-AQFM, U8 TCA9548AMRGER, U9 760308101214

Commit message: 5V
Parts:
- removed C7: 10uF, Footprints:GRM21BR60J226ME39L, symbol Symbols:GRM21BZ71E106KE15L
- added C19, C20: 22uF, GRM31x, symbol Symbols:GRM31CZ71C226ME15L
- added R17: 7.87k, ERJU01_(0201), symbol Symbols:ERJU01F7871C
Connections:
- net 1.2V: now also U10.4 (AVIN), U10.5 (PVIN), C20.1
- net GND: now also U10.3 (GND), C19.2, C20.2
- net at U10.1 (VSEL): now also R17.1
- net +5V: now reaches U10.2 (VOUT)
- net +5V: now also C19.1
- net U10_7: now reaches U10.7 (EN)
- no-connect marks 20 -> 21
Other:
- moved on the sheet: U10

Commit message: begin 1.8V, 1.9V, 3.3V, 4.5V + fixups
Parts:
- added C21, C22, C28: 22uF, GRM31x, symbol Symbols:GRM31CZ71C226ME15L
- added C69, C7: 10uF, GRM21BR60J226ME39L, symbol Symbols:GRM21BZ71E106KE15L
- added IC8, IC9: TPS7A9601DSCR, TPS7A9601DSCR, symbol Symbols:TPS7A9601DSCR
- added R18: 7.87k, ERJU01_(0201), symbol Symbols:ERJU01F7871C
- added U21: TPSM81299VCMR, VCM0007A-MFG, symbol Symbols:TPSM81299VCMR
Connections:
- net +1.9V: now also C69.2, IC9.1 (IN_1)
- net +3.3V: now also C22.1, U21.2 (VOUT)
- net +5V: now also C7.2, IC8.1 (IN_1)
- net 1.2V: now also U21.4 (AVIN), U21.5 (PVIN)
- net GND: now also R17.2, C21.2, C22.2, C28.2, C69.1, C7.1, IC8.6 (GND), R18.2, U21.3 (GND)
- net U10_7: now also U21.7 (EN)
- new net: R18.1, U21.1 (VSEL)
- new net +1.8V: C28.1, IC9.9 (OUT_1)
- new net +4.5V: C21.1, IC8.9 (OUT_1)
- no-connect marks 21 -> 24
Other:
- note added: "TPS7A96_1"
- note added: "TPS7A96_2"
- moved on the sheet: BT1, C1, C10, C11, C12, C13, C15, C16, C17, C19, C2, C20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

Commit message: power
Parts:
- removed R18: 7.87k, ERJU01_(0201), symbol Symbols:ERJU01F7871C
- added C70: 10uF, GRM21BR60J226ME39L, symbol Symbols:GRM21BZ71E106KE15L
- added C71: 1uF, GRM155R61H334ME01D, symbol Symbols:GRM155D71E105KE11J
- added C72: 2.2uF, GRM18x, symbol Symbols:GRM188Z71E225KE43J
- added R18: 30k, ERJU01_(0201), symbol Symbols:ERJU01F3002C
- added R19: 30k, ERJU01_(0201), symbol Symbols:ERJU01F1202C
- added R20, R21, R26: 10k, ERJU01_(0201), symbol Symbols:ERJU01J103C
- added R22, R24: 12.7k, ERJU01_(0201), symbol Symbols:ERJU01F1272C
- added R23: 240k, ERJU01_(0201), symbol Symbols:ERJU01F2403C
- added R25: 90.9k, ERJU01_(0201), symbol Symbols:ERJU01F9092C
- added R27, R28: 1M, ERJU01_(0201), symbol Symbols:ERJU01F1004C
- added R_{NTC}2: 10K, Footprints:ERTJ0EA101H, symbol Symbols:ERTJ0EG103FA
Connections:
- net PACK+ is gone; now on net VSS: BT1.1 (+), C6.1, IC2.C2 (BAT), U3.6 (VBACKUP)
- net +1.8V: now also IC9.10 (OUT_2), IC9.8 (SNS), C70.1, R25.2
- net +1.9V: now also IC9.2 (IN_2), R20.2
- net +4.5V: now also IC8.10 (OUT_2), R23.2
- net +5V: now also IC8.2 (IN_2), R21.2
- net 1.2V: no longer C20.1, IC2.B2 (SYS), U10.4 (AVIN), U10.5 (PVIN), U21.4 (AVIN), U21.5 (PVIN)
- net GND: now also IC9.6 (GND), U21.1 (VSEL), C70.2, C71.2, R18.2, R19.2, R22.1, R24.1, R_{NTC}2.2
- net VSS: now also C20.1, IC2.B2 (SYS), U10.4 (AVIN), U10.5 (PVIN), U21.4 (AVIN), U21.5 (PVIN), U5.C2 (SRX), U5.C3 (BAT), C71.1, C72.2, R26.2, R27.2, R28.2
- net at U5.A1 (GPOUT): now also R26.1
- net at U5.A2 (SDA): now also R27.1
- net at U5.A3 (SCL): now also R28.1
- net at U5.B1 (BIN): now also R_{NTC}2.1
- net at U5.B3 (VDD): now also C72.1
- net at IC8.4 (PG): now also R21.1
- net at IC8.5 (FB_PG): now also R22.2, R23.1
- net at IC8.7 (NR/SS): now also R18.1
- net at IC9.4 (PG): now also R20.1
- net at IC9.5 (FB_PG): now also R24.2, R25.1
- net at IC9.7 (NR/SS): now also R19.1
- no-connect marks 24 -> 33
Other:
- moved on the sheet: C28, U5

Commit message: correct typos + begin AS7058
Parts:
- removed C6: 1uF, Footprints:CAPC3216X95N, symbol Symbols:GRM3195C1H103FA01D
- removed C71: 1uF, GRM155R61H334ME01D, symbol Symbols:GRM155D71E105KE11J
- removed R19: 30k, ERJU01_(0201), symbol Symbols:ERJU01F1202C
- removed U1: AS7058, symbol Symbols:AS7058
- added C73, C74: 1uF, GRM155R61H334ME01D, symbol Symbols:GRM155D71E105KE11J
- added R19: 30k, ERJU01_(0201), symbol Symbols:ERJU01F3002C
- added U1: AS7058, symbol AS7058:AS7058
- LNA_EN1: value MAX-M10S -> MAX-M10S (Switch to M11 once released)
- U12: value BMI270 -> BMI270 (Switch to BMI570 once released)
Connections:
- net +1.8V: now also U1.F1 (AVDD2), U1.G4 (AVDD1)
- net +4.5V: now also U1.C2 (VCSELS)
- net GND: now also C73.2, C74.2, R19.2
- net VSS: now also C73.1, C74.1
- net at IC9.7 (NR/SS): now also R19.1
- new net: U1.F2 (AGND2), U1.G5 (AGND1)
Other:
- note removed: "Sensors"
- moved on the sheet: IC3
