File: KiCad/LibrePulse.kicad_sch (KiCad schematic)
At the start: 202 parts, among them IC1 AS6221, IC10 BME690, IC11 KLMCG4JETD-B041, IC2 TPS62841YBGR, IC3 BQ21088YBGR, IC4 TPS62840YBGR, IC5 OPT3007YMFR, IC6 ICU-10201, IC7 TPS7A9601DSCR, IC8 TPS7A9601DSCR, IC9 TPS62840YBGR, J1 SIDE_CROWN_PAD2, J2 ECG_INP_PAD, J3 ECG_REF_PAD, J4 SIDE_CROWN_PAD1, J5 Micro_SD_Card, M1 VLV041235L, U1 AS7058, U10 TPSM81299VCMR, U11 TPSM81299VCMR, U12 BMI270, U13 BMM350, U14 DRV2605LDGS, U15 ET020AM03-HT, U16 LM3643YFFR, U17 CXD5610GF, U18 ESP32-C6, U19 HP5354.A, U2 RV-3028-C8-32.768KHZ-1PPM-TA-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, U20 TPS7A5701RTER, U21 BGA524N6, U22 TPS7A5701RTER, U23 BGA524N6, U3 W25Q128JVS, U4 MS5837-30BA, U5 BQ51013CQWRHLRQ1, U6 BQ27427YZFR, U7 PCAL6416AHF, U8 ESP32-P4NRW32, U9 760308101214, Y1 WE-SPXO_CFPS-39, Y2 ECS-TXO-20CSMV4-260-AN-TR, Y3 ECS-TXO-20CSMV4-260-AN-TR

Commit message: initial stuff I did yesterday but forgot today
Parts:
- removed D1, D2, D20, D21, D3, D4, D5, D6: SFH 7018, Footprints:SMD8_2p4x2p4_SFH7018A_OSM, symbol Device:D
- removed D10, D11, D13, D15, D16, D7, D8, D9: SFH 2202, OptoDevice:Osram_SFH2201, symbol Device:D_Photo
- added D1, D2, D3, D4, D5, D6, D7, D8: SFH2705U, SFH2705U, symbol Symbols:SFH2705U
- added IC12: AD5940BCBZ-RL, BGA56C40P8X7_416X356X55, symbol Symbols:AD5940BCBZ-RL
- added LED2, LED3: SFH_7019, SFH7019, symbol Symbols:SFH_7019
- added LED4: SFH_7014H, SFH7014H, symbol Symbols:SFH_7014H
Connections:
- net +4V5: now also LED2.2 (IR._UV_(ANODE)_1), LED2.5 (IR._UV_(ANODE)_2), LED2.6 (G_(ANODE)), LED3.2 (IR._UV_(ANODE)_1), LED3.5 (IR._UV_(ANODE)_2), LED3.6 (G_(ANODE)), LED4.2 (ANODE_BLUE/_GREEN/_RED/_IR_EMITTER_1), LED4.5 (ANODE_BLUE/_GREEN/_RED/_IR_EMITTER_2)
- net LED1: now also LED2.4 (UV_(CATHODE))
- net LED2: now also LED3.4 (UV_(CATHODE))
- net LED3: now also LED2.3 (G_(CATHODE))
- net LED4: now also LED3.3 (G_(CATHODE))
- net LED5: now also LED2.1 (IR_(CATHODE))
- net LED6: now also LED3.1 (IR_(CATHODE))
- net LED7: now also LED4.4 (CATHODE_RED_EMITTER_(655_NM))
- net LED8: now also LED4.6 (CATHODE_BLUE_EMITTER_(460_NM))
- net PDREF: now also D1.1 (K), D2.1 (K), D3.1 (K), D4.1 (K), D5.1 (K), D6.1 (K), D7.1 (K), D8.1 (K)
- net at U1.F4 (PD3): now also D6.2 (A)
- net at U1.E3 (PD8): now also D1.2 (A)
- net at U1.D3 (PD6): now also D3.2 (A)
- net at U1.D4 (PD4): now also D5.2 (A)
- net at U1.G3 (PD2): now also D7.2 (A)
- net at U1.E4 (PD1): now also D8.2 (A)
- net at U1.F3 (PD7): now also D2.2 (A)
- net at U1.G2 (PD5): now also D4.2 (A)
- no-connect marks 234 -> 236
Other:
- moved on the sheet: C16, C27, C28, C34, C36, C37, C40, C41, C42, C43, C49, C50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

Commit message: begin optimizing power by replacing with MAX77826 + cleanups
Parts:
- removed ANT1: W3008, Footprints:ANTENNA_W3008, symbol Symbols:W3008
- removed ANT2: HC125A, HC125A, symbol Symbols:HC125A
- removed BT1: DTP793435-1S1P-1300mAh-3.85V, Connector_PinHeader_2.54mm:PinHeader_1x02_P2.54mm_Vertical, symbol Device:Battery_Cell
- removed C1, C13, C2, C3, C65: 1uF, Footprints:GRM155R61H334ME01D, symbol Symbols:GRM155D71E105KE11J
- removed C10, C11, C15, C25, C47, C48, C5, C51, C52, C66, C67: 10uF, Footprints:GRM21BR60J226ME39L, symbol Symbols:GRM21BZ71E106KE15L
- removed C12, C7: 2.2uF, Footprints:GRM18x, symbol Symbols:GRM188Z71E225KE43J
- removed C14, C53, C6: 4.7uF, Footprints:GRM21BR60J226ME39L, symbol Symbols:GRM21BZ71E475KE15L
- removed C17: 100pF, Footprints:GRM033D70J224ME01D, symbol Symbols:GRM0335C1H102GE01J
- removed C18, C33: 22nF, Footprints:CAPC2012X145N, symbol Symbols:GRM21B5C1H223FA01L
- removed C19, C26: 10nF, Footprints:CAPC3216X95N, symbol Symbols:GRM3195C1H103FA01D
- removed C20, C24: 100nF, Footprints:GRMJN65C1H104JE01D, symbol Symbols:GRMJN65C1H104GE01D
- removed C21, C22, C31, C32: 47nF, Footprints:CAPC3216X95N, symbol Symbols:GRM3195C1H103FA01D
- removed C23: 1nF, Footprints:GRM033D70J224ME01D, symbol Symbols:GRM0335C1H102GE01J
- removed C29, C30, C44, C45, C8: 22uF, Footprints:GRM31x, symbol Symbols:GRM31CZ71C226ME15L
- removed C34, C36, C37, C38, C4, C46, C54, C58, C59, C61, C76, C77, C9: 100nF, Footprints:GRM033D70J224ME01D, symbol Symbols:GRM033Z71C104KE14J
- removed C35, C39: 470nF, Footprints:CAPC3216X180N, symbol Symbols:GRM31C5C1E474GE01K
- removed C57: 2.2uF, Footprints:CAPC2212X200N, symbol Symbols:KRM21FD71H225KFA1L
- removed C60: 47pF, Footprints:GRM033D70J224ME01D, symbol Symbols:GJM1555C1H470FB01J
- removed C69, C71: 4.7uF, GRM21BR60J226ME39L, symbol Symbols:GRM21BZ71E475KE15L
- removed D1, D2, D3, D4, D5, D6, D7, D8: SFH2705U, SFH2705U, symbol Symbols:SFH2705U
- removed D12, D14, D17, D19: PESD5V0V1BL, Footprints:DIO_PESD5V5C1ULYL, symbol Device:D_TVS
- removed FL1: QPQ1060TR7, QPQ1060TR7, symbol Symbols:QPQ1060TR7
- removed FL2: B39122B7505L210, B39122B7505L210, symbol Symbols:B39122B7505L210
- removed IC1: AS6221, Footprints:BGA6C40P3X2_149X102X60, symbol Symbols:AS6221
- removed IC10: BME690, Footprints:BME690, symbol Symbols:BME690
- removed IC11: KLMCG4JETD-B041, Footprints:BGA153C50P14X14_1150X1300X80, symbol Symbols:KLMAG1JETD-B041
- removed IC12: AD5940BCBZ-RL, BGA56C40P8X7_416X356X55, symbol Symbols:AD5940BCBZ-RL
- removed IC2: TPS62841YBGR, Footprints:BGA6C40P2X3_97X147X50, symbol Symbols:TPS62841YBGR
- removed IC3: BQ21088YBGR, Footprints:BGA8C40P2X4_100X155X50, symbol Symbols:BQ21088YBGR
- removed IC4, IC9: TPS62840YBGR, Footprints:BGA6C40P2X3_97X147X50, symbol Symbols:TPS62840YBGR
- removed IC5: OPT3007YMFR, Footprints:BGA6C35P2X3_86X95X23, symbol Symbols:OPT3007YMFR
- removed IC6: ICU-10201, Footprints:ICU10201, symbol Symbols:ICU-10201
- removed IC7, IC8: TPS7A9601DSCR, Footprints:TPS7A9601DSCR, symbol Symbols:TPS7A9601DSCR
- removed J1: SIDE_CROWN_PAD2, TestPoint:TestPoint_Pad_D2.0mm, symbol Connector_Generic:Conn_01x01
- removed J2: ECG_INP_PAD, TestPoint:TestPoint_Pad_D2.0mm, symbol Connector_Generic:Conn_01x01
- removed J3: ECG_REF_PAD, TestPoint:TestPoint_Pad_D2.0mm, symbol Connector_Generic:Conn_01x01
- removed J4: SIDE_CROWN_PAD1, TestPoint:TestPoint_Pad_D2.0mm, symbol Connector_Generic:Conn_01x01
- removed J5: Micro_SD_Card, Connector_Card:microSD_HC_Wuerth_693072010801, symbol Connector:Micro_SD_Card
- removed L1, L2, L3: 2.2uH, Footprints:744777002, symbol Symbols:744777002
- removed L4: 1uH, Footprints:INDC1608X80N, symbol Symbols:74479262210
- removed L5, L6: 8.2nH, WE-TCI_040286, symbol Symbols:744901082
- removed LED1: KW_CSLPM1.TG-8N7P-EBVF46FCBB46, Footprints:KWCSLNM1TG8M7NebvF46fcbB4615B5, symbol Symbols:KW_CSLPM1.TG-8N7P-EBVF46FCBB46
- removed LED2, LED3: SFH_7019, SFH7019, symbol Symbols:SFH_7019
- removed LED4: SFH_7014H, SFH7014H, symbol Symbols:SFH_7014H
- removed M1: VLV041235L, Haptic_Motors:VLV041235L, symbol Motor:Motor_DC
- removed R1, R3, R5, R6: 10K, Footprints:ERJU01__0201_, symbol Symbols:ERJU01J103C
- removed R10, R9: 33, Footprints:ERJU01__0201_, symbol Symbols:ERJU01J330C
- removed R11, R16, R18, R19: 1M, Footprints:ERJU01__0201_, symbol Symbols:ERJU01F1004C
- removed R12, R17: 51k, Footprints:ERJU01__0201_, symbol Symbols:ERJU01F1004C
- removed R13: 196, Footprints:ERJU01__0201_, symbol Symbols:ERJU01F1960C
- removed R15, R33, R34, R41, R42, R45, R48, R49, R50, R51: 10k, Footprints:ERJU01__0201_, symbol Symbols:ERJU01J103C
- removed R2, R7, R8: 47k, Footprints:ERJ2RKD1004X, symbol Symbols:ERJ2RKF4702X
- removed R20, R21, R26, R27: 100k, Footprints:ERJU01__0201_, symbol Symbols:ERJU01J104C
- removed R23, R24, R28, R29: 5.1k, Footprints:ERJU01__0201_, symbol Symbols:ERJU01F1004C
- removed R25: 1.5k, Footprints:ERJU01__0201_, symbol Symbols:ERJU01J152C
- removed R30: 7.87k, Footprints:ERJU01__0201_, symbol Symbols:ERJU01F7871C
- removed R31: 11.5k, Footprints:ERJU01__0201_, symbol Symbols:ERJU01F1152C
- removed R32, R35: 30k, Footprints:ERJU01__0201_, symbol Symbols:ERJU01F3002C
- removed R36, R38: 12.7k, Footprints:ERJU01__0201_, symbol Symbols:ERJU01F1272C
- removed R37: 240k, Footprints:ERJU01__0201_, symbol Symbols:ERJU01F2403C
- removed R39: 90.9k, Footprints:ERJU01__0201_, symbol Symbols:ERJU01F9092C
- removed R4: 16k, Footprints:ERJU01__0201_, symbol Symbols:ERJU01F1602C
- removed R40: 10k, Footprints:ERJS02_U02__0402_, symbol Symbols:ERJU02F1002X
- removed R43: 10k, ERJS02_U02_(0402), symbol Symbols:ERJU02F1002X
- removed R44, R47: 4.7k, Footprints:ERJ2RKD1004X, symbol Symbols:ERJ2RKF4702X
- removed R52: 16k, ERJU01_(0201), symbol Symbols:ERJU01F1602C
- removed R53, R54: 100, Footprints:ERJU01__0201_, symbol Symbols:ERJU02F1002X
- removed R_{NTC}1, R_{NTC}2: 10K, Footprints:ERTJ0EA101H, symbol Symbols:ERTJ0EG103FA
- removed U1: AS7058, AS7058:BGA-42_6x7_2.55x2.82mm, symbol AS7058:AS7058
- removed U10, U11: TPSM81299VCMR, Footprints:VCM0007A-MFG, symbol Symbols:TPSM81299VCMR
- removed U12: BMI270, Footprints:BMI270, symbol Symbols:BMI270
- removed U13: BMM350, Footprints:BMM350, symbol Symbols:BMM350
- removed U14: DRV2605LDGS, Package_SO:TSSOP-10_3x3mm_P0.5mm, symbol Driver:DRV2605LDGS
- removed U16: LM3643YFFR, Footprints:IC_LM3643YFFR, symbol Symbols:LM3643YFFR
- removed U17: CXD5610GF, symbol CXD5610GF:CXD5610GF
- removed U18: ESP32-C6, Footprints:ESP32-C6, symbol Symbols:ESP32-C6
- removed U19: HP5354.A, symbol HP5354.A:HP5354.A
- removed U2: RV-3028-C8-32.768KHZ-1PPM-TA-QC, Footprints:RV-3028-C8-32.768KHZ-1PPM-TA-QC, symbol RV-3028-C8-32.768KHZ-1PPM-TA-QC:RV-3028-C8-32.768KHZ-1PPM-TA-QC
- removed U20, U22: TPS7A5701RTER, WQFN16_RTE_TEX, symbol Symbols:TPS7A5701RTER
- removed U21, U23: BGA524N6, BGA524N6:INF-PG-TSNP-6-2-V, symbol Symbols:BGA524N6
- removed U4: MS5837-30BA, Sensor_Pressure:TE_MS5837-xxBA, symbol Sensor_Pressure:MS5837-xxBA
- removed U5: BQ51013CQWRHLRQ1, Footprints:IC_BQ51013CQWRHLRQ1, symbol Symbols:BQ51013CQWRHLRQ1
- removed U6: BQ27427YZFR, Footprints:BQ27427YZFR, symbol Symbols:BQ27427YZFR
- removed U9: 760308101214, Footprints:760308101214, symbol Symbols:760308101214
- removed Y1: WE-SPXO_CFPS-39, Footprints:WE-SPXO_CFPS-39, symbol Symbols:WE-SPXO_CFPS-39
- removed Y2, Y3: ECS-TXO-20CSMV4-260-AN-TR, ECS-TXO-20CSMV4-260-AN-TR:OSC_ECS-TXO-20CSMV4-260-AN-TR, symbol Symbols:ECS-TXO-20CSMV4-260-AN-TR
Connections:
- no-connect marks 236 -> 53
Other:
- note removed: "BQ21088"
- note removed: "BQ27427YZFR"
- note removed: "BQ51013CQWRHLRQ1"
- note removed: "Battery"
- note removed: "Connectivity"
- note removed: "GNSS"
- note removed: "Light"
- note removed: "Note: Switch to BMI570 once released"
- note removed: "Power"
- note removed: "RV-3028-C8"
- note removed: "Random Shit"
- note removed: "Storage"
- note removed: "TPS62840YBGR"
- note removed: "TPS62841YBGR"
- note removed: "TPS7A96_1"
- note removed: "TPS7A96_2"
- note removed: "TPSM81299"

Commit message: Begin Initial Redesign and Cleanup
Parts:
- removed C16, C27, C28, C40, C41, C49, C50: 100nF, Footprints:GRM033D70J224ME01D, symbol Symbols:GRM033Z71C104KE14J
- removed C42, C43, C55, C56: 10uF, Footprints:GRM21BR60J226ME39L, symbol Symbols:GRM21BZ71E106KE15L
- removed R14: 10kΩ, Footprints:ERJU01__0201_, symbol Symbols:ERJU02F1002X
- removed R22: 10k, Footprints:ERJS02_U02__0402_, symbol Symbols:ERJU02F1002X
- removed U3: W25Q128JVS, Package_SO:SOIC-8_5.3x5.3mm_P1.27mm, symbol Memory_Flash:W25Q128JVS
- removed U7: PCAL6416AHF, Package_DFN_QFN:HVQFN-24-1EP_4x4mm_P0.5mm_EP2.1x2.1mm, symbol Interface_Expansion:PCAL6416AHF
- removed U8: ESP32-P4NRW32, Footprints:ESP32-P4NRW32, symbol ESP32-P4NRW32:ESP32-P4NRW32
- added U1: STM32U599NJHxQ, Package_BGA:TFBGA-216_13x13mm_Layout15x15_P0.8mm, symbol MCU_ST_STM32U5:STM32U599NJHxQ
Connections:
- new net: U1.A1 (VSS), U1.A15 (VSS), U1.E10 (VSS), U1.F10 (VSS), U1.F6 (VSS), U1.F7 (VSS), U1.F9 (VSS), U1.G10 (VSS), U1.H10 (VSS), U1.H15 (VSS), U1.J10 (VSS), U1.J15 (VSS), U1.J6 (VSS), U1.K10 (VSS), U1.K7 (VSS), U1.K8 (VSS), U1.K9 (VSS), U1.L10 (VSS), U1.R1 (VSS), U1.R15 (VSS)
- new net: U1.G6 (VSSDSI), U1.H2 (VSSDSI), U1.H6 (VSSDSI), U1.J2 (VSSDSI)
- no-connect marks 53 -> 10
Other:
- note removed: "MCU"

Commit message: cleanup and continue redesign
Parts:
- removed U1: STM32U599NJHxQ, Package_BGA:TFBGA-216_13x13mm_Layout15x15_P0.8mm, symbol MCU_ST_STM32U5:STM32U599NJHxQ
- added U1: MIMXRT758SGFOB, symbol MIMXRT758SGFOB:MIMXRT758SGFOB
Other:
- moved on the sheet: C62, C63, C64, C68, U15

Commit message: redesign
Parts:
- removed U1: MIMXRT758SGFOB, symbol MIMXRT758SGFOB:MIMXRT758SGFOB
- added IC13: AP510BFA-CBR, BGA153C40P13X13_560X560X80, symbol Symbols:AP510BFA-CBR
- added IC8: AKD1500PFC040BA, BGA169C50P13X13_700X700X130, symbol Symbols:AKD1500PFC040BA
