File: KiCad/misc._sensors.kicad_sch (KiCad schematic)
At the start: 8 parts, among them IC10 SHT40-AD1B-R2, M1 VLV041235L, U14 DRV2605LDGS, U3 BMP581

Commit message: continue redesign
Parts:
- added LS1: AST-01508MR-R, AST-01508MR-R:SPKR_AST-01508MR-R, symbol Symbols:AST-01508MR-R
- added MK1: IM69D130, Sensor_Audio:Infineon_PG-LLGA-5-1, symbol Sensor_Audio:IM69D130
- added U11: MAX98357A, Package_DFN_QFN:TQFN-16-1EP_3x3mm_P0.5mm_EP1.23x1.23mm, symbol Audio:MAX98357A
Connections:
- new net: U11.11 (GND), U11.15 (GND), U11.3 (GND)
- new net: U11.7 (VDD), U11.8 (VDD)

Commit message: cleanup and continue redesign
Parts:
- removed U3: BMP581, BMP581, symbol Symbols:BMP581
- added A1: BMP585, BMP585:XDCR_BMP585, symbol Symbols:BMP585
Connections:
- net GND: no longer C60.2, R40.2, U14.8 (GND)
- new net GNDD: C60.2, R40.2, U14.8 (GND)
