File: KiCad/motion.kicad_sch (KiCad schematic)
At the start: 3 parts, among them IC6 ICU-10201, IC7 LSM6DSO16IS, IC9 IIS2MDCTR

Commit message: continue redesign
Changed lines of the file:
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@@
 	(generator_version "10.0")
 	(paper "A4")
-	(label "SPI{SCK,MOSI,MISO,CS}"
-		(at 80.01 149.86 0)
-		(effects
-			(font
-				(size 1.27 1.27)
-			)
-			(justify left bottom)
-		)
-	)
 	(symbol
 		(lib_id "Symbols:ICU-10201")

Commit message: cleanup and continue redesign
Parts:
- removed IC7: LSM6DSO16IS, Footprints:LSM6DSV16BXTR, symbol Symbols:LSM6DSO16IS
- added IC7: LSM6DSV80XTR, LSM6DSV16BXTR, symbol Symbols:LSM6DSV80XTR
Connections:
- net GNDD: now reaches IC6.1 (GND_1)
- net GNDD: now also IC6.11 (GND_3), IC6.8 (GND_2)
- new net +1V8: IC7.5 (VDDIO), IC7.8 (VDD)
- new net GND: IC7.13 (SCL), IC7.14 (SDA), IC7.6 (GND_1), IC7.7 (GND_2)
- no-connect marks 0 -> 2
