File: KiCad/power.kicad_sch (KiCad schematic)
At the start: 37 parts, among them IC2 MAX77826EWJ+T, IC3 BQ21088YBGR, U2 RV-3028-C8-32.768KHZ-1PPM-TA-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, U5 BQ51013CQWRHLRQ1, U6 BQ27427YZFR, U9 760308101214

Commit message: cleanup and continue redesign
Parts:
- removed IC2: MAX77826EWJ+T, BGA49C40P7X7_302X302X69, symbol Symbols:MAX77826EWJ+T
- added IC4: MAX77714FEWC+T, BGA70C40P10X7_412X317X69, symbol Symbols:MAX77714FEWC+T
- added U10: MAX77827AEFD, Package_DFN_QFN:Maxim_FC2QFN-14_2.5x2.5mm_P0.5mm, symbol Regulator_Switching:MAX77827AEFD
- added U8: TPS7A20xxxDBV, Package_TO_SOT_SMD:SOT-23-5, symbol Regulator_Linear:TPS7A20xxxDBV
Connections:
- net U6_14 is gone; now on net AC2: U5.19 (AC2)
- net U6_2 is gone; now on net AC1: U5.2 (AC1)
- net GND: no longer BT1.2 (-), C10.1, C13.2, C15.1, C24.2, C25.2, C7.2, C8.2, C9.1, IC3.D2 (GND), R10.2, R13.2, R6.2, R9.1, R_{NTC}1.2, R_{NTC}2.2, U5.1 (PGND), U5.12 (ILIM), U5.20 (PGND), U5.21 (EXP), U5.9 (AD)
- net AC1: now reaches C23.1, C26.1, C33.1, C39.1, U9.2
- net AC1: now also U5.3 (BOOT1), U5.5 (CLAMP1), U5.6 (COMM1); no longer C35.1
- net GNDPWR: now reaches C39.2
- net GNDPWR: now also BT1.2 (-), C10.1, C13.2, C15.1, C18.2, C19.2, C24.2, C25.2, C26.2, C33.2, C35.2, C7.2, C8.2, C9.1, IC3.D2 (GND), R10.2, R13.2, R6.2, R9.1, R_{NTC}1.2, R_{NTC}2.2, U5.1 (PGND), U5.12 (ILIM), U5.20 (PGND), U5.21 (EXP), U5.9 (AD)
- net AC2: now reaches U5.15 (COMM2)
- net AC2: now also C18.1, C19.1, C20.1, C23.2, C35.1, U5.16 (CLAMP2), U5.17 (BOOT2)
- new net: U10.4 (PGND), U10.9 (PGND)
Other:
- moved on the sheet: C10, C15, C18, C19, C20, C23, C26, C33, C39, C9, U9

Commit message: redesign
Other:
- moved on the sheet: U10
Changed lines of the file:
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@@
 	(symbol
 		(lib_id "Regulator_Switching:MAX77827AEFD")
-		(at 430.53 137.16 0)
+		(at 402.59 143.51 0)
 		(unit 1)
 		(body_style 1)
@@
 		(fields_autoplaced yes)
 		(property "Reference" "U10"
-			(at 430.53 121.92 0)
+			(at 402.59 128.27 0)
 			(show_name no)
 			(do_not_autoplace no)
@@
 		)
 		(property "Value" "MAX77827AEFD"
-			(at 430.53 124.46 0)
+			(at 402.59 130.81 0)
 			(show_name no)
 			(do_not_autoplace no)
@@
 		)
 		(property "Footprint" "Package_DFN_QFN:Maxim_FC2QFN-14_2.5x2.5mm_P0.5mm"
-			(at 430.53 123.19 0)
+			(at 402.59 129.54 0)
 			(hide yes)
 			(show_name no)
@@
 		)
 		(property "Datasheet" "https://www.analog.com/media/en/technical-documentation/data-sheets/MAX77827.pdf"
-			(at 430.53 120.65 0)
+			(at 402.59 127 0)
 			(hide yes)
 			(show_name no)
@@
 		)
 		(property "Description" "5.5V Input, 1.8A/3.1A Switch Buck-Boost, QFN-14"
-			(at 430.53 137.16 0)
+			(at 402.59 143.51 0)
 			(hide yes)
 			(show_name no)
