File: KiCad/storage.kicad_sch (KiCad schematic)
At the start: 3 parts, among them IC11 KLMCG4JETD-B041, J5 Micro_SD_Card

Commit message: cleanup and continue redesign
Connections:
- net GND: no longer IC11.A6 (VSS_1), IC11.C4 (VSS_2), IC11.E7 (VSS_3), IC11.G5 (VSS_4), IC11.H10 (VSS_5), IC11.J5 (VSS_6), IC11.K8 (VSS_7), IC11.N2 (VSS_8), IC11.N5 (VSS_9), IC11.P4 (VSS_10), IC11.P6 (VSS_11)
- new net GNDD: IC11.A6 (VSS_1), IC11.C4 (VSS_2), IC11.E7 (VSS_3), IC11.G5 (VSS_4), IC11.H10 (VSS_5), IC11.K8 (VSS_7), IC11.N5 (VSS_9), IC11.P4 (VSS_10), IC11.P6 (VSS_11)

Commit message: redesign
Parts:
- removed C65: 1uF, Footprints:GRM155R61H334ME01D, symbol Symbols:GRM155D71E105KE11J
- removed IC11: KLMCG4JETD-B041, Footprints:BGA153C50P14X14_1150X1300X80, symbol Symbols:KLMAG1JETD-B041
- removed J5: Micro_SD_Card, Connector_Card:microSD_HC_Wuerth_693072010801, symbol Connector:Micro_SD_Card
- added IC11: UFS64G-CY14-02N01, BGA153C50P14X14_1100X1300X85, symbol Symbols:UFS64G-CY14-02N01
Connections:
- no-connect marks 122 -> 0

Commit message: aaaa
Parts:
- removed IC11: UFS64G-CY14-02N01, BGA153C50P14X14_1100X1300X85, symbol Symbols:UFS64G-CY14-02N01
- added IC11: KLMAG1JETD-B041, BGA153C50P14X14_1150X1300X80, symbol Symbols:KLMAG1JETD-B041
