File: KiCad/connectivity.kicad_sch (KiCad schematic)
At the start: 28 parts, among them IC17 GM02SP, U11 MAX98357A, U17 CXD5610GF, U18 ESP32-C6, U19 HP5354.A, U21 BGA524N6, U23 BGA524N6, Y1 WE-SPXO_CFPS-39, Y3 ECS-TXO-20CSMV4-260-AN-TR

Commit message: continue redesign
Parts:
- removed ANT1: W3008, Footprints:ANTENNA_W3008, symbol Symbols:W3008
- removed C76, C77: 100nF, Footprints:GRM033D70J224ME01D, symbol Symbols:GRM033Z71C104KE14J
- removed IC17: GM02SP, Footprints:GM02SP, symbol Symbols:GM02SP
- removed R41, R42, R45, R48, R49, R50, R51: 10k, Footprints:ERJU01__0201_, symbol Symbols:ERJU01J103C
- removed U18: ESP32-C6, Footprints:ESP32-C6, symbol Symbols:ESP32-C6
- removed Y1: WE-SPXO_CFPS-39, Footprints:WE-SPXO_CFPS-39, symbol Symbols:WE-SPXO_CFPS-39
- added IC1: NRF7002-QFAA-R7, QFN40P600X600X95-49N, symbol Symbols:NRF7002-QFAA-R7
- added IC12: NRF54L15-QFAA-R, QFN40P600X600X95-49N, symbol Symbols:NRF54L15-QFAA-R
- added IC2: SARA-R410M-02B, SARAR412M02B, symbol Symbols:SARA-R410M-02B
Connections:
- no-connect marks 30 -> 6

Commit message: continue redesign
Parts:
- removed LS1: AST-01508MR-R, AST-01508MR-R:SPKR_AST-01508MR-R, symbol Symbols:AST-01508MR-R
- removed MK1: IM69D130, Sensor_Audio:Infineon_PG-LLGA-5-1, symbol Sensor_Audio:IM69D130
- removed U11: MAX98357A, Package_DFN_QFN:TQFN-16-1EP_3x3mm_P0.5mm_EP1.23x1.23mm, symbol Audio:MAX98357A

Commit message: cleanup and continue redesign
Changed lines of the file:
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@@
 		(at 62.23 105.41)
+	)
+	(bus_entry
+		(at 154.94 29.21)
+		(size 2.54 2.54)
+		(stroke
+			(width 0)
+			(type default)
+		)
 	)
 	(wire

Commit message: redesign
Other:
- note removed: "GNSS"
Changed lines of the file:
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@@
 	(generator_version "10.0")
 	(paper "A3")
-	(text "GNSS"
-		(exclude_from_sim no)
-		(at 116.332 40.894 0)
-		(effects
-			(font
-				(size 6.35 6.35)
-			)
-		)
-	)
 	(junction
 		(at 64.77 73.66)

Commit message: update
Parts:
- removed IC12: NRF54L15-QFAA-R, QFN40P600X600X95-49N, symbol Symbols:NRF54L15-QFAA-R
Other:
- moved on the sheet: IC2

Commit message: aaaa
Other:
- moved on the sheet: IC2
Changed lines of the file:
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@@
 	(symbol
 		(lib_id "Symbols:SARA-R410M-02B")
-		(at 265.43 100.33 0)
+		(at 180.34 123.19 0)
 		(unit 1)
 		(body_style 1)
@@
 		(fields_autoplaced yes)
 		(property "Reference" "IC2"
-			(at 290.83 92.71 0)
+			(at 205.74 115.57 0)
 			(show_name no)
 			(do_not_autoplace no)
@@
 		)
 		(property "Value" "SARA-R410M-02B"
-			(at 290.83 95.25 0)
+			(at 205.74 118.11 0)
 			(show_name no)
 			(do_not_autoplace no)
@@
 		)
 		(property "Footprint" "SARAR412M02B"
-			(at 312.42 195.25 0)
+			(at 227.33 218.11 0)
 			(hide yes)
 			(show_name no)
@@
 		)
 		(property "Datasheet" "https://www.u-blox.com/sites/default/files/SARA-R4-N4_DataSheet_%28UBX-16024152%29.pdf"
-			(at 312.42 295.25 0)
+			(at 227.33 318.11 0)
 			(hide yes)
 			(show_name no)
@@
 		)
 		(property "Description" "Size-optimized LTE Cat M1/NB1 and EGPRS modules"
-			(at 265.43 100.33 0)
+			(at 180.34 123.19 0)
 			(hide yes)
 			(show_name no)
@@
 		)
 		(property "Height" "2.53"
-			(at 312.42 495.25 0)
+			(at 227.33 518.11 0)
 			(hide yes)
 			(show_name no)
@@
 		)
 		(property "Manufacturer_Name" "u-blox"
-			(at 312.42 595.25 0)
+			(at 227.33 618.11 0)
 			(hide yes)
 			(show_name no)
@@
 		)
 		(property "Manufacturer_Part_Number" "SARA-R410M-02B"
-			(at 312.42 695.25 0)
+			(at 227.33 718.11 0)
 			(hide yes)
 			(show_name no)
@@
 		)
 		(property "Mouser Part Number" "377-SARA-R410M-02B"
-			(at 312.42 795.25 0)
+			(at 227.33 818.11 0)
 			(hide yes)
 			(show_name no)
@@
 		)
 		(property "Mouser Price/Stock" "https://www.mouser.co.uk/ProductDetail/u-blox/SARA-R410M-02B?qs=DPoM0jnrROWddJ2vKHR9ag%3D%3D"
-			(at 312.42 895.25 0)
+			(at 227.33 918.11 0)
 			(hide yes)
 			(show_name no)
@@
 		)
 		(property "Arrow Part Number" "SARA-R410M-02B"
-			(at 312.42 995.25 0)
+			(at 227.33 1018.11 0)
 			(hide yes)
 			(show_name no)
@@
 		)
 		(property "Arrow Price/Stock" "https://www.arrow.com/en/products/sara-r410m-02b/u-blox?utm_currency=USD&region=nac"
-			(at 312.42 1095.25 0)
+			(at 227.33 1118.11 0)
 			(hide yes)
 			(show_name no)

Commit message: simplify
Parts:
- removed IC1: NRF7002-QFAA-R7, QFN40P600X600X95-49N, symbol Symbols:NRF7002-QFAA-R7
Other:
- moved on the sheet: IC2, U17
