File: KiCad/health.kicad_sch (KiCad schematic)
At the start: 15 parts, among them IC1 AS6221, IC4 ADPD4200BCBZR7, IC8 ADPD4200BCBZR7, U10 ADGS6414DBCCZ, U20 ADGS6414DBCCZ, U22 ADGS6414DBCCZ, U24 ADGS6414DBCCZ

Commit message: cleanup and continue redesign
Parts:
- removed IC1: AS6221, Footprints:BGA6C40P3X2_149X102X60, symbol Symbols:AS6221
- removed IC4, IC8: ADPD4200BCBZR7, Footprints:BGA24C40P4X6_180X262X57, symbol Symbols:ADPD4200BCBZR7
- removed U10, U20, U22, U24: ADGS6414DBCCZ, Footprints:CC-30-3_ADI, symbol Symbols:ADGS6414DBCCZ
- added IC14: AS6223A-AWLT, AS6223AAWLT, symbol Symbols:AS6223A-AWLT
- added U3, U4: ADPD7000BCBZR7, CB-36-11_ADI, symbol Symbols:ADPD7000BCBZR7
- added U7: ADPD4100BCBZR7, CB-35-2_ADI, symbol Symbols:ADPD4100BCBZR7

Commit message: simplify
Parts:
- removed LED12, LED13: SFH_7019, Footprints:SFH7019, symbol Symbols:SFH_7019
- removed LED14, LED15: LO_R976-PS-1, Footprints:LEDC2012X90N, symbol Symbols:LO_R976-PS-1
- removed LED16, LED17: LY_R976-PS-36, LEDC2013X90N, symbol Symbols:LY_R976-PS-36
- removed U3, U4: ADPD7000BCBZR7, CB-36-11_ADI, symbol Symbols:ADPD7000BCBZR7
- removed U7: ADPD4100BCBZR7, CB-35-2_ADI, symbol Symbols:ADPD4100BCBZR7
- added U1: AS7058, symbol AS7058:AS7058
Other:
- moved on the sheet: IC14
